File: electrical/HP_classic.sch (KiCad schematic (older format))
At the start: 15 parts, among them J1 USB_B_Micro, J2 JST PH 2mm, J3 2.54mm R/A, U1 MCP73831-2-OT

Commit message: Version 1 Checkin
Schematic updated with component details
PCB udpated for plot formatting
Check plots generated
Interactive BOM generated
Parts:
- C1, C2: DigiKey (none) -> 490-14466-1-ND; MPN (none) -> MuRata GRM21BR71C475KE51L; WVDC (none) -> 16V
- D1: Color (none) -> RED
- J1: DigiKey (none) -> WM10134CT-ND; MPN (none) -> Molex 1051330011
- J2: DigiKey (none) -> 455-1719-ND; MPN (none) -> S2B-PH-K-S(LF)(SN)
- U1: DigiKey (none) -> MCP73831T-2ACI/OTCT-ND; MPN (none) -> Microchip MCP73831T-2ACI/OT
Changed lines of the file:
@@
 F 2 "Package_TO_SOT_SMD:SOT-23-5" H 4700 3350 50  0001 L CIN
 F 3 "http://ww1.microchip.com/downloads/en/DeviceDoc/20001984g.pdf" H 4500 3550 50  0001 C CNN
+F 4 "Microchip MCP73831T-2ACI/OT" H 4650 3600 50  0001 C CNN "MPN"
+F 5 "MCP73831T-2ACI/OTCT-ND" H 4650 3600 50  0001 C CNN "DigiKey"
 	1    4650 3600
 	1    0    0    -1
@@
 F 2 "Connector_USB:USB_Micro-B_Molex-105133-0001" H 2650 3350 50  0001 C CNN
 F 3 "~" H 2650 3350 50  0001 C CNN
+F 4 "Molex 1051330011" H 2500 3400 50  0001 C CNN "MPN"
+F 5 "WM10134CT-ND" H 2500 3400 50  0001 C CNN "DigiKey"
 	1    2500 3400
 	1    0    0    -1
@@
 F 2 "Capacitor_SMD:C_0805_2012Metric" H 3600 3700 50  0001 C CNN
 F 3 "~" H 3600 3700 50  0001 C CNN
+F 4 "16V" H 3750 3550 50  0000 C CNN "WVDC"
+F 5 "MuRata GRM21BR71C475KE51L" H 3600 3700 50  0001 C CNN "MPN"
+F 6 "490-14466-1-ND" H 3600 3700 50  0001 C CNN "DigiKey"
 	1    3600 3700
 	1    0    0    -1
@@
 	1    0    0    -1
 $EndComp
-$Comp
-L Device:C_Small C2
-U 1 1 5FA3C240
-P 6000 3700
-F 0 "C2" H 6092 3746 50  0000 L CNN
-F 1 "4.7uF" H 6092 3655 50  0000 L CNN
-F 2 "Capacitor_SMD:C_0805_2012Metric" H 6000 3700 50  0001 C CNN
-F 3 "~" H 6000 3700 50  0001 C CNN
-	1    6000 3700
-	1    0    0    -1
-$EndComp
 Wire Wire Line
 	6000 3600 6000 3200
@@
 F 2 "Connector_JST:JST_PH_S2B-PH-K_1x02_P2.00mm_Horizontal" H 6700 3700 50  0001 C CNN
 F 3 "~" H 6700 3700 50  0001 C CNN
+F 4 "S2B-PH-K-S(LF)(SN)" H 6700 3700 50  0001 C CNN "MPN"
+F 5 "455-1719-ND" H 6700 3700 50  0001 C CNN "DigiKey"
 	1    6700 3700
 	1    0    0    -1
@@
 F 3 "~" H 5500 3950 50  0001 C CNN
 F 4 "CHARGE" V 5402 3832 50  0000 R CNN "Function"
+F 5 "RED" V 5500 3950 50  0001 C CNN "Color"
 	1    5500 3950
 	0    -1   -1   0
@@
 Text Notes 3750 4800 0    75   ~ 0
 R1 = 5.1K sets\n200mA CC
+$Comp
+L Device:C_Small C2
+U 1 1 5FB54FB6
+P 6000 3700
+F 0 "C2" H 6092 3746 50  0000 L CNN
+F 1 "4.7uF" H 6092 3655 50  0000 L CNN
+F 2 "Capacitor_SMD:C_0805_2012Metric" H 6000 3700 50  0001 C CNN
+F 3 "~" H 6000 3700 50  0001 C CNN
+F 4 "16V" H 6150 3550 50  0000 C CNN "WVDC"
+F 5 "MuRata GRM21BR71C475KE51L" H 6000 3700 50  0001 C CNN "MPN"
+F 6 "490-14466-1-ND" H 6000 3700 50  0001 C CNN "DigiKey"
+	1    6000 3700
+	1    0    0    -1
+$EndComp
 $EndSCHEMATC
